Commit message: badly works via gui publisher

File: module_3_assignment/urdf/tf_tree.urdf (robot description, URDF)
Before this commit: robot tf_tree, 3 links, 3 joints
Links:
- added link link_3, mass 0.5; collision cylinder length=0.5 radius=0.05; visual cylinder length=0.5 radius=0.05
- link base_link: geometry collision box size=0.2 0.2 0.1; visual box size=0.2 0.2 0.1
- link link_1: mass None -> 0.5; geometry collision cylinder length=0.5 radius=0.05; visual cylinder length=0.5 radius=0.05
- link link_2: mass None -> 0.5; geometry collision cylinder length=0.5 radius=0.05; visual cylinder length=0.5 radius=0.05
Joints:
- removed joint base_joint
- added joint joint_3: type revolute, parent link_2, child link_3, origin xyz=0.25 0.0 0.0 rpy=0.0 0.0 0.0, axis 0.0 0.0 1.0, limit lower=-1.57 upper=1.57 effort=1.0 velocity=1.0
- joint joint_1: axis 0.0 1.0 0.0 -> 0.0 0.0 1.0; child link_2 -> link_1; limit lower=-3.14 upper=3.14 effort=1.0 velocity=0.0 -> lower=-1.57 upper=1.57 effort=1.0 velocity=1.0; origin xyz=0.0 0.0 0.48 rpy=0.0 0.0 0.0 -> xyz=0.1 0.0 0.05 rpy=0.0 0.0 0.0; parent link_1 -> base_link; type fixed -> revolute
- joint joint_2: axis 0.0 1.0 0.0 -> 0.0 0.0 1.0; limit lower=-3.14 upper=3.14 effort=1.0 velocity=0.0 -> lower=-1.57 upper=1.57 effort=1.0 velocity=1.0; origin xyz=0.0 1.0 0.48 rpy=0.0 0.0 0.0 -> xyz=0.25 0.0 0.0 rpy=0.0 0.0 0.0; type fixed -> revolute

Commit message: well works via gui publisher

File: module_3_assignment/urdf/tf_tree.urdf (robot description, URDF)
Before this commit: robot three_link_robot, 4 links, 3 joints
Links:
- removed link link_3
- added link gripper
- link base_link: geometry 
- link link_1: mass 0.5 -> None; geometry 
- link link_2: mass 0.5 -> None; geometry 
Joints:
- removed joint joint_3
- added joint base_joint: type continuous, parent base_link, child link_1, origin xyz=0.0 0.0 0.0 rpy=0.0 0.0 0.0, axis 0.0 0.0 1.0
- joint joint_1: axis 0.0 0.0 1.0 -> 0.0 1.0 0.0; child link_1 -> link_2; limit lower=-1.57 upper=1.57 effort=1.0 velocity=1.0 -> lower=-3.14 upper=3.14 effort=1.0 velocity=0.0; origin xyz=0.1 0.0 0.05 rpy=0.0 0.0 0.0 -> xyz=0.0 0.0 1.48 rpy=0.0 0.0 0.0; parent base_link -> link_1
- joint joint_2: child link_2 -> gripper; limit lower=-1.57 upper=1.57 effort=1.0 velocity=1.0 -> lower=-3.14 upper=3.14 effort=1.0 velocity=0.0; origin xyz=0.25 0.0 0.0 rpy=0.0 0.0 0.0 -> xyz=0.0 0.0 1.48 rpy=0.0 0.0 0.0; parent link_1 -> link_2
