Commit message: task_3 pre-complited

File: module_3_assignment/urdf/static_robot.urdf (robot description, URDF)
Before this commit: robot tf_tree, 6 links, 5 joints
Links:
- removed link base_link
- removed link finger_1
- removed link finger_2
- removed link gripper
- removed link link_1
- removed link link_2
Joints:
- removed joint base_joint
- removed joint joint_1
- removed joint joint_2
- removed joint joint_3
- removed joint joint_4
