Commit message: task_3 complited

File: module_3_assignment/urdf/combined_robot.urdf (robot description, URDF)
Before this commit: robot combined_robot, 9 links, 8 joints
Links:
- removed link wheel_left
- removed link wheel_right
- added link camera, mass 0.1; collision box size=0.1 0.1 0.05; visual box size=0.1 0.1 0.05
- added link caster, mass 1; collision sphere radius=.08; visual sphere radius=.08
- added link lidar, mass 0.5; collision box size=0.1 0.1 0.1; visual cylinder length=0.05 radius=0.1
- added link wheel_left_link, mass 2; collision cylinder length=0.1 radius=0.15; visual cylinder length=0.1 radius=0.15
- added link wheel_right_link, mass 2; collision cylinder length=0.1 radius=0.15; visual cylinder length=0.1 radius=0.15
- link mobile_base: mass None -> 1; geometry collision box size=0.75 0.4 0.1; visual box size=0.75 0.4 0.1
Joints:
- added joint camera_joint: type fixed, parent mobile_base, child camera, origin xyz=-0.35 0 0.01 rpy=0 0.0 3.14, axis 0.0 0.0 1.0
- added joint caster_joint: type continuous, parent mobile_base, child caster, origin xyz=-0.3 0.0 -0.07 rpy=0.0 0.0 0.0, axis 0 0 1
- added joint lidar_joint: type fixed, parent mobile_base, child lidar, origin xyz=-0.285 0 0.075 rpy=0 0.0 1.57, axis 0.0 0.0 1.0
- joint wheel_left_joint: axis 0 1 0 -> 0.0 0.0 1.0; child wheel_left -> wheel_left_link; origin xyz=-0.3 0.2 0.1 rpy=0 0 0 -> xyz=0.2 -0.25 0.0 rpy=1.57 0.0 0.0
- joint wheel_right_joint: axis 0 1 0 -> 0.0 0.0 1.0; child wheel_right -> wheel_right_link; origin xyz=-0.3 -0.2 0.1 rpy=0 0 0 -> xyz=0.2 0.25 0.0 rpy=1.57 0.0 0.0

File: module_3_assignment/urdf/combo_bot.xacro (robot description, xacro)
@@ -5,5 +5,5 @@
     <xacro:mobile_robot base_link="mobile_base"/>
     <joint name="connector_joint" type="fixed">
-        <origin xyz="0.0 0.0 0.0" rpy="0.0 0.0 0.0"/>
+        <origin xyz="0.0 0.0 3.0" rpy="0.0 0.0 0.0"/>
         <parent link="mobile_base"/>
         <child link="base_link"/>

File: module_3_assignment/urdf/mobile_robot.xacro (robot description, xacro)
@@ -3,63 +3,170 @@
     <xacro:macro name="mobile_robot" params="base_link">
     <!-- Базовая платформа -->
-    <link name="${base_link}">
-        <visual>
-            <geometry>
-                <box size="0.6 0.4 0.2"/>
-            </geometry>
-            <material name="red">
-                <color rgba="1.0 0.0 0.0 1.0"/>
-            </material>
-        </visual>
-        <collision>
-            <geometry>
-                <box size="0.6 0.4 0.2"/>
-            </geometry>
-        </collision>
-    </link>
-    <!-- Колеса -->
-    <link name="wheel_left">
-        <visual>
-            <geometry>
-                <cylinder radius="0.05" length="0.02"/>
-            </geometry>
-            <material name="black">
-                <color rgba="0.0 0.0 0.0 1.0"/>
-            </material>
-        </visual>
-        <collision>
-            <geometry>
-                <cylinder radius="0.05" length="0.02"/>
-            </geometry>
-        </collision>
-    </link>
-    <link name="wheel_right">
-        <visual>
-            <geometry>
-                <cylinder radius="0.05" length="0.02"/>
-            </geometry>
-            <material name="black">
-                <color rgba="0.0 0.0 0.0 1.0"/>
-            </material>
-        </visual>
-        <collision>
-            <geometry>
-                <cylinder radius="0.05" length="0.02"/>
-            </geometry>
-        </collision>
-    </link>
-    <!-- Шарниры для колес -->
-    <joint name="wheel_left_joint" type="continuous">
-        <origin xyz="-0.3 0.2 0.1" rpy="0 0 0"/>
-        <parent link="${base_link}"/>
-        <child link="wheel_left"/>
-        <axis xyz="0 1 0"/>
-    </joint>
-    <joint name="wheel_right_joint" type="continuous">
-        <origin xyz="-0.3 -0.2 0.1" rpy="0 0 0"/>
-        <parent link="${base_link}"/>
-        <child link="wheel_right"/>
-        <axis xyz="0 1 0"/>
-    </joint>
+     <link name="${base_link}">
+    <visual>
+      <geometry>
+          <box size="0.75 0.4 0.1"/>
+      </geometry>
+      <material name="gray">
+        <color rgba=".2 .2 .2 1" />
+      </material>
+    </visual>
+    <inertial>
+        <mass value="1" />
+        <inertia ixx="0.01" ixy="0.0" ixz="0" iyy="0.01" iyz="0" izz="0.01" />
+    </inertial>
+    <collision>
+      <geometry>
+          <box size="0.75 0.4 0.1"/>
+      </geometry>
+    </collision>
+  </link>
+  <link name="wheel_right_link">
+    <inertial>
+            <mass value="2" />
+            <inertia ixx="0.01" ixy="0.0" ixz="0"
+            iyy="0.01" iyz="0" izz="0.01" />
+    </inertial>
+    <visual>
+      <geometry>
+          <cylinder radius="0.15" length="0.1"/>
+      </geometry>
+      <material name="white">
+        <color rgba="1 1 1 1"/>
+      </material>
+    </visual>
+    <collision>
+      <geometry>
+          <cylinder radius="0.15" length="0.1"/>
+      </geometry>
+      <contact_coefficients mu="1" kp="1e+13" kd="1.0"/>
+    </collision>
+  </link>
+  <joint name="wheel_right_joint" type="continuous">
+    <origin xyz="0.2 0.25 0.0" rpy="1.57 0.0 0.0"/>
+    <parent link="${base_link}"/>
+    <child link="wheel_right_link"/>
+    <axis xyz="0.0 0.0 1.0"/>
+  </joint>
+  <link name="wheel_left_link">
+    <inertial>
+            <mass value="2" />
+            <inertia ixx="0.01" ixy="0.0" ixz="0"
+            iyy="0.01" iyz="0" izz="0.01" />
+    </inertial>
+    <visual>
+      <geometry>
+          <cylinder radius="0.15" length="0.1"/>
+      </geometry>
+      <material name="white">
+        <color rgba="1 1 1 1"/>
+      </material>
+    </visual>
+    <collision>
+      <geometry>
+          <cylinder radius="0.15" length="0.1"/>
+      </geometry>
+      <contact_coefficients mu="1" kp="1e+13" kd="1.0"/>
+    </collision>
+  </link>
+  <joint name="wheel_left_joint" type="continuous">
+    <origin xyz="0.2 -0.25 0.0" rpy="1.57 0.0 0.0"/>
+    <parent link="${base_link}"/>
+    <child link="wheel_left_link"/>
+    <axis xyz="0.0 0.0 1.0"/>
+  </joint>
+  <link name="caster">
+    <inertial>
+            <mass value="1" />
+            <inertia ixx="0.01" ixy="0.0" ixz="0"
+            iyy="0.01" iyz="0" izz="0.01" />
+    </inertial>
+    <visual>
+      <geometry>
+        <sphere radius=".08" />
+      </geometry>
+      <material name="white" />
+    </visual>
+    <collision>
+      <origin/>
+      <geometry>
+        <sphere radius=".08" />
+      </geometry>
+    </collision>
+  </link>
+  <joint name="caster_joint" type="continuous">
+    <origin xyz="-0.3 0.0 -0.07" rpy="0.0 0.0 0.0"/>
+    <axis xyz="0 0 1" />
+    <parent link="${base_link}"/>
+    <child link="caster"/>
+  </joint>
+  <link name="camera">
+    <inertial>
+            <mass value="0.1" />
+            <inertia ixx="0.01" ixy="0.0" ixz="0"
+            iyy="0.01" iyz="0" izz="0.01" />
+    </inertial>
+    <visual>
+      <geometry>
+        <box size="0.1 0.1 0.05"/>
+      </geometry>
+      <material name="white">
+        <color rgba="1 1 1 1"/>
+      </material>
+    </visual>
+    <collision>
+      <geometry>
+          <box size="0.1 0.1 0.05"/>
+      </geometry>
+    </collision>
+  </link>
+  <joint name="camera_joint" type="fixed">
+    <origin xyz="-0.35 0 0.01" rpy="0 0.0 3.14"/>
+    <parent link="${base_link}"/>
+    <child link="camera"/>
+    <axis xyz="0.0 0.0 1.0"/>
+  </joint>
+  <link name="lidar">
+    <inertial>
+            <mass value="0.5" />
+            <inertia ixx="0.01" ixy="0.0" ixz="0"
+            iyy="0.01" iyz="0" izz="0.01" />
+    </inertial>
+    <visual>
+      <geometry>
+        <cylinder radius="0.1" length="0.05"/>
+      </geometry>
+      <material name="white">
+        <color rgba="1 1 1 1"/>
+      </material>
+    </visual>
+    <collision>
+      <geometry>
+          <box size="0.1 0.1 0.1"/>
+      </geometry>
+    </collision>
+  </link>
+  <joint name="lidar_joint" type="fixed">
+    <origin xyz="-0.285 0 0.075" rpy="0 0.0 1.57"/>
+    <parent link="${base_link}"/>
+    <child link="lidar"/>
+    <axis xyz="0.0 0.0 1.0"/>
+  </joint>
+  <gazebo>
+    <plugin filename="libgazebo_ros_diff_drive.so" name="gazebo_base_controller">
+      <odometry_frame>odom</odometry_frame>
+      <commandTopic>cmd_vel</commandTopic>
+      <publish_odom>true</publish_odom>
+      <publish_odom_tf>true</publish_odom_tf>
+      <update_rate>15.0</update_rate>
+      <left_joint>wheel_left_joint</left_joint>
+      <right_joint>wheel_right_joint</right_joint>
+      <wheel_separation>0.5</wheel_separation>
+      <wheel_diameter>0.3</wheel_diameter>
+      <max_wheel_acceleration>0.7</max_wheel_acceleration>
+      <max_wheel_torque>8</max_wheel_torque>
+      <robotBaseFrame>base</robotBaseFrame>
+    </plugin>
+  </gazebo>
     </xacro:macro>
 </robot>
