Commit message: task_3 complited with pure xacro and launch

File: module_3_assignment/urdf/combo_bot.xacro (robot description, xacro)
@@ -5,5 +5,5 @@
     <xacro:mobile_robot base_link="mobile_base"/>
     <joint name="connector_joint" type="fixed">
-        <origin xyz="0.0 0.0 3.0" rpy="0.0 0.0 0.0"/>
+        <origin xyz="0.0 0.0 0.1" rpy="0.0 0.0 0.0"/>
         <parent link="mobile_base"/>
         <child link="base_link"/>

Commit message: task_3 akkerman v1

File: module_3_assignment/urdf/combo_bot.xacro (robot description, xacro)
@@ -3,8 +3,8 @@
     <!-- Включение мобильной платформы -->
     <xacro:include filename="mobile_robot.xacro"/>
-    <xacro:mobile_robot base_link="mobile_base"/>
+    <xacro:mobile_robot base_link="chassis"/>
     <joint name="connector_joint" type="fixed">
         <origin xyz="0.0 0.0 0.1" rpy="0.0 0.0 0.0"/>
-        <parent link="mobile_base"/>
+        <parent link="chassis"/>
         <child link="base_link"/>
         <axis xyz="0.0 0.0 1.0"/>

File: module_3_assignment/urdf/mobile_robot.xacro (robot description, xacro)
@@ -2,171 +2,127 @@
 <robot xmlns:xacro="http://www.ros.org/wiki/xacro" name="mobile_robot">
     <xacro:macro name="mobile_robot" params="base_link">
-    <!-- Базовая платформа -->
-     <link name="${base_link}">
+  <link name="${base_link}">
     <visual>
       <geometry>
-          <box size="0.75 0.4 0.1"/>
+        <box size="1.0 0.5 0.2"/>
       </geometry>
-      <material name="gray">
-        <color rgba=".2 .2 .2 1" />
-      </material>
-    </visual>
-    <inertial>
-        <mass value="1" />
-        <inertia ixx="0.01" ixy="0.0" ixz="0" iyy="0.01" iyz="0" izz="0.01" />
-    </inertial>
-    <collision>
-      <geometry>
-          <box size="0.75 0.4 0.1"/>
-      </geometry>
-    </collision>
-  </link>
-  <link name="wheel_right_link">
-    <inertial>
-            <mass value="2" />
-            <inertia ixx="0.01" ixy="0.0" ixz="0"
-            iyy="0.01" iyz="0" izz="0.01" />
-    </inertial>
-    <visual>
-      <geometry>
-          <cylinder radius="0.15" length="0.1"/>
-      </geometry>
-      <material name="white">
-        <color rgba="1 1 1 1"/>
+      <material name="blue">
+        <color rgba="0.0 0.0 1.0 1.0"/>
       </material>
     </visual>
     <collision>
       <geometry>
-          <cylinder radius="0.15" length="0.1"/>
+        <box size="1.0 0.5 0.2"/>
       </geometry>
-      <contact_coefficients mu="1" kp="1e+13" kd="1.0"/>
     </collision>
   </link>
-  <joint name="wheel_right_joint" type="continuous">
-    <origin xyz="0.2 0.25 0.0" rpy="1.57 0.0 0.0"/>
-    <parent link="${base_link}"/>
-    <child link="wheel_right_link"/>
-    <axis xyz="0.0 0.0 1.0"/>
-  </joint>
-  <link name="wheel_left_link">
-    <inertial>
-            <mass value="2" />
-            <inertia ixx="0.01" ixy="0.0" ixz="0"
-            iyy="0.01" iyz="0" izz="0.01" />
-    </inertial>
+  <!-- Передние колеса -->
+  <link name="front_left_wheel">
     <visual>
+    <origin xyz="0.0 0.0 0.0" rpy="1.56 0.0 0.0"/>
       <geometry>
-          <cylinder radius="0.15" length="0.1"/>
+        <cylinder length="0.1" radius="0.15"/>
       </geometry>
-      <material name="white">
-        <color rgba="1 1 1 1"/>
+      <material name="black">
+        <color rgba="0.0 0.0 0.0 1.0"/>
       </material>
     </visual>
     <collision>
+    <origin xyz="0.0 0.0 0.0" rpy="1.56 0.0 0.0"/>
       <geometry>
-          <cylinder radius="0.15" length="0.1"/>
-      </geometry>
-      <contact_coefficients mu="1" kp="1e+13" kd="1.0"/>
-    </collision>
-  </link>
-  <joint name="wheel_left_joint" type="continuous">
-    <origin xyz="0.2 -0.25 0.0" rpy="1.57 0.0 0.0"/>
-    <parent link="${base_link}"/>
-    <child link="wheel_left_link"/>
-    <axis xyz="0.0 0.0 1.0"/>
-  </joint>
-  <link name="caster">
-    <inertial>
-            <mass value="1" />
-            <inertia ixx="0.01" ixy="0.0" ixz="0"
-            iyy="0.01" iyz="0" izz="0.01" />
-    </inertial>
-    <visual>
-      <geometry>
-        <sphere radius=".08" />
-      </geometry>
-      <material name="white" />
-    </visual>
-    <collision>
-      <origin/>
-      <geometry>
-        <sphere radius=".08" />
+        <cylinder length="0.1" radius="0.15"/>
       </geometry>
     </collision>
   </link>
-  <joint name="caster_joint" type="continuous">
-    <origin xyz="-0.3 0.0 -0.07" rpy="0.0 0.0 0.0"/>
-    <axis xyz="0 0 1" />
-    <parent link="${base_link}"/>
-    <child link="caster"/>
-  </joint>
-  <link name="camera">
-    <inertial>
-            <mass value="0.1" />
-            <inertia ixx="0.01" ixy="0.0" ixz="0"
-            iyy="0.01" iyz="0" izz="0.01" />
-    </inertial>
+  <link name="front_right_wheel">
     <visual>
+    <origin xyz="0.0 0.0 0.0" rpy="1.56 0.0 0.0"/>
       <geometry>
-        <box size="0.1 0.1 0.05"/>
+        <cylinder length="0.1" radius="0.15"/>
       </geometry>
-      <material name="white">
-        <color rgba="1 1 1 1"/>
+      <material name="black">
+        <color rgba="0.0 0.0 0.0 1.0"/>
       </material>
     </visual>
     <collision>
+    <origin xyz="0.0 0.0 0.0" rpy="1.56 0.0 0.0"/>
       <geometry>
-          <box size="0.1 0.1 0.05"/>
+        <cylinder length="0.1" radius="0.15"/>
       </geometry>
     </collision>
   </link>
-  <joint name="camera_joint" type="fixed">
-    <origin xyz="-0.35 0 0.01" rpy="0 0.0 3.14"/>
-    <parent link="${base_link}"/>
-    <child link="camera"/>
-    <axis xyz="0.0 0.0 1.0"/>
-  </joint>
-  <link name="lidar">
-    <inertial>
-            <mass value="0.5" />
-            <inertia ixx="0.01" ixy="0.0" ixz="0"
-            iyy="0.01" iyz="0" izz="0.01" />
-    </inertial>
+  <!-- Задние колеса -->
+  <link name="rear_left_wheel">
     <visual>
+    <origin xyz="0.0 0.0 0.0" rpy="1.56 0.0 0.0"/>
       <geometry>
-        <cylinder radius="0.1" length="0.05"/>
+        <cylinder length="0.1" radius="0.15"/>
       </geometry>
-      <material name="white">
-        <color rgba="1 1 1 1"/>
+      <material name="black">
+        <color rgba="0.0 0.0 0.0 1.0"/>
       </material>
     </visual>
     <collision>
+    <origin xyz="0.0 0.0 0.0" rpy="1.56 0.0 0.0"/>
       <geometry>
-          <box size="0.1 0.1 0.1"/>
+        <cylinder length="0.1" radius="0.15"/>
       </geometry>
     </collision>
   </link>
-  <joint name="lidar_joint" type="fixed">
-    <origin xyz="-0.285 0 0.075" rpy="0 0.0 1.57"/>
+  <link name="rear_right_wheel">
+    <visual>
+    <origin xyz="0.0 0.0 0.0" rpy="1.56 0.0 0.0"/>
+      <geometry>
+        <cylinder length="0.1" radius="0.15"/>
+      </geometry>
+      <material name="black">
+        <color rgba="0.0 0.0 0.0 1.0"/>
+      </material>
+    </visual>
+    <collision>
+    <origin xyz="0.0 0.0 0.0" rpy="1.56 0.0 0.0"/>
+      <geometry>
+        <cylinder length="0.1" radius="0.15"/>
+      </geometry>
+    </collision>
+  </link>
+  <!-- Шарниры для передних колес -->
+  <joint name="front_left_steering_joint" type="revolute">
     <parent link="${base_link}"/>
-    <child link="lidar"/>
-    <axis xyz="0.0 0.0 1.0"/>
+    <child link="front_left_wheel"/>
+    <origin xyz="0.4 0.3 -0.265" rpy="0 0 0"/>
+    <axis xyz="0 0 1"/>
+    <limit lower="-0.5" upper="0.5" effort="1.0" velocity="1.0"/>
+  </joint>
+  <joint name="front_right_steering_joint" type="revolute">
+    <parent link="${base_link}"/>
+    <child link="front_right_wheel"/>
+    <origin xyz="0.4 -0.3 -0.265" rpy="0 0 0"/>
+    <axis xyz="0 0 1"/>
+    <limit lower="-0.5" upper="0.5" effort="1.0" velocity="1.0"/>
+  </joint>
+  <!-- Шарниры для вращения колес -->
+  <joint name="rear_left_drive_joint" type="continuous">
+    <parent link="${base_link}"/>
+    <child link="rear_left_wheel"/>
+    <origin xyz="-0.4 0.3 -0.265" rpy="0 0 0"/>
+    <axis xyz="0 1 0"/>
+  </joint>
+  <joint name="rear_right_drive_joint" type="continuous">
+    <parent link="${base_link}"/>
+    <child link="rear_right_wheel"/>
+    <origin xyz="-0.4 -0.3 -0.265" rpy="0 0 0"/>
+    <axis xyz="0 1 0"/>
   </joint>
   <gazebo>
-    <plugin filename="libgazebo_ros_diff_drive.so" name="gazebo_base_controller">
-      <odometry_frame>odom</odometry_frame>
-      <commandTopic>cmd_vel</commandTopic>
-      <publish_odom>true</publish_odom>
-      <publish_odom_tf>true</publish_odom_tf>
-      <update_rate>15.0</update_rate>
-      <left_joint>wheel_left_joint</left_joint>
-      <right_joint>wheel_right_joint</right_joint>
-      <wheel_separation>0.5</wheel_separation>
-      <wheel_diameter>0.3</wheel_diameter>
-      <max_wheel_acceleration>0.7</max_wheel_acceleration>
-      <max_wheel_torque>8</max_wheel_torque>
-      <robotBaseFrame>base</robotBaseFrame>
-    </plugin>
-  </gazebo>
+  <plugin name="ackermann_steering_plugin" filename="libackermann_steering_plugin.so">
+    <left_steering_joint>front_left_steering_joint</left_steering_joint>
+    <right_steering_joint>front_right_steering_joint</right_steering_joint>
+    <left_drive_joint>rear_left_drive_joint</left_drive_joint>
+    <right_drive_joint>rear_right_drive_joint</right_drive_joint>
+    <wheel_base>1.0</wheel_base>
+    <track_width>0.6</track_width>
+  </plugin>
+</gazebo>
     </xacro:macro>
 </robot>
