Commit message: task_3 akkerman v1.1

File: module_3_assignment/urdf/mobile_robot.xacro (robot description, xacro)
@@ -17,4 +17,39 @@
     </collision>
   </link>
+<!--steering links-->
+<link name="left_steering">
+    <inertial>
+        <origin xyz="0.0 0.0 0.0" rpy="0.0 0.0 0.0"/>
+        <mass value="0.0"/>
+        <!-- <inertia ixx="0.0" ixy="0.0" ixz="0.0" iyy="0.0" iyz="0.0" izz="0.0"/> -->
+    </inertial>
+    <visual name="">
+        <origin xyz="0.0 0.0 0.0" rpy="0.0 0.0 0.0"/>
+        <geometry>
+            <cylinder length="0.04" radius="0.01"/>
+        </geometry>
+        <material name="">
+            <color rgba="1.0 0.0 0.0 1.0"/>
+            <texture filename=""/>
+        </material>
+    </visual>
+</link>
+<link name="right_steering">
+    <inertial>
+        <origin xyz="0.0 0.0 0.0" rpy="0.0 0.0 0.0"/>
+        <mass value="0.0"/>
+        <!-- <inertia ixx="0.0" ixy="0.0" ixz="0.0" iyy="0.0" iyz="0.0" izz="0.0"/> -->
+    </inertial>
+    <visual name="">
+        <origin xyz="0.0 0.0 0.0" rpy="0.0 0.0 0.0"/>
+        <geometry>
+            <cylinder length="0.04" radius="0.01"/>
+        </geometry>
+        <material name="">
+            <color rgba="1.0 0.0 0.0 1.0"/>
+            <texture filename=""/>
+        </material>
+    </visual>
+</link>
   <!-- Передние колеса -->
   <link name="front_left_wheel">
@@ -87,8 +122,8 @@
     </collision>
   </link>
-  <!-- Шарниры для передних колес -->
+  <!-- Шарниры для поворота колес -->
   <joint name="front_left_steering_joint" type="revolute">
     <parent link="${base_link}"/>
-    <child link="front_left_wheel"/>
+    <child link="left_steering"/>
     <origin xyz="0.4 0.3 -0.265" rpy="0 0 0"/>
     <axis xyz="0 0 1"/>
@@ -97,8 +132,21 @@
   <joint name="front_right_steering_joint" type="revolute">
     <parent link="${base_link}"/>
-    <child link="front_right_wheel"/>
+    <child link="right_steering"/>
     <origin xyz="0.4 -0.3 -0.265" rpy="0 0 0"/>
     <axis xyz="0 0 1"/>
     <limit lower="-0.5" upper="0.5" effort="1.0" velocity="1.0"/>
+  </joint>
+<!--шарниры для вращения колёс-->
+  <joint name="front_left_wheel_joint" type="continuous">
+    <parent link="left_steering"/>
+    <child link="front_left_wheel"/>
+    <origin xyz="-0.4 0.3 -0.265" rpy="0 0 0"/>
+    <axis xyz="0 1 0"/>
+  </joint>
+  <joint name="front_right_wheel_joint" type="continuous">
+    <parent link="right_steering"/>
+    <child link="front_right_wheel"/>
+    <origin xyz="-0.4 -0.3 -0.265" rpy="0 0 0"/>
+    <axis xyz="0 1 0"/>
   </joint>
   <!-- Шарниры для вращения колес -->

Commit message: task_3 akkerman v1.1

File: module_3_assignment/urdf/mobile_robot.xacro (robot description, xacro)
@@ -141,5 +141,5 @@
     <parent link="left_steering"/>
     <child link="front_left_wheel"/>
-    <origin xyz="-0.4 0.3 -0.265" rpy="0 0 0"/>
+    <origin xyz="0 0 0" rpy="0 0 0"/>
     <axis xyz="0 1 0"/>
   </joint>
@@ -147,5 +147,5 @@
     <parent link="right_steering"/>
     <child link="front_right_wheel"/>
-    <origin xyz="-0.4 -0.3 -0.265" rpy="0 0 0"/>
+    <origin xyz="0 0 0" rpy="0 0 0"/>
     <axis xyz="0 1 0"/>
   </joint>

Commit message: task_3 akkerman v1.5

File: module_3_assignment/urdf/mobile_robot.xacro (robot description, xacro)
@@ -22,5 +22,5 @@
         <origin xyz="0.0 0.0 0.0" rpy="0.0 0.0 0.0"/>
         <mass value="0.0"/>
-        <!-- <inertia ixx="0.0" ixy="0.0" ixz="0.0" iyy="0.0" iyz="0.0" izz="0.0"/> -->
+        <inertia ixx="0.0" ixy="0.0" ixz="0.0" iyy="0.0" iyz="0.0" izz="0.0"/>
     </inertial>
     <visual name="">
@@ -39,5 +39,5 @@
         <origin xyz="0.0 0.0 0.0" rpy="0.0 0.0 0.0"/>
         <mass value="0.0"/>
-        <!-- <inertia ixx="0.0" ixy="0.0" ixz="0.0" iyy="0.0" iyz="0.0" izz="0.0"/> -->
+        <inertia ixx="0.0" ixy="0.0" ixz="0.0" iyy="0.0" iyz="0.0" izz="0.0"/>
     </inertial>
     <visual name="">
